File: crank/sensor2/sensor2.kicad_pcb (KiCad board)
At the start: 2 copper layers, 25.4 x 25.4 mm, 5 parts, among them J3 Conn_01x04_Socket, U1 TLV493D

Commit message: cleanup
Other:
- board text added: "Playdate Cabinet Crank Sensor 2"
- board text removed: "Playdate Cabinet Crank Sensor 2 2024.10.3 dave@ panic.com"
