File: crank/sensor2/sensor2.kicad_sch (KiCad schematic)
At the start: 5 parts, among them J3 Conn_01x04_Socket, U1 TLV493D

Commit message: cleanup
Changed lines of the file:
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@@
 (kicad_sch
-	(version 20231120)
+	(version 20250114)
 	(generator "eeschema")
-	(generator_version "8.0")
+	(generator_version "9.0")
 	(paper "A4")
 	(junction
@@
 		)
 	)
+	(embedded_fonts no)
 )
